File: Hardware/PCBModels/ArduinoShieldDesign/CEWBPCBDesign.kicad_pcb (KiCad board)
At the start: 2 copper layers, 95.6 x 65 mm, 6 parts

Commit message: Updated PCB Design
Parts:
- added JP1: Jumper_2_Bridged, Resistor_THT:R_Axial_DIN0204_L3.6mm_D1.6mm_P5.08mm_Horizontal, F.Cu at (163.0, 95.9)
- added JP2: Jumper_2_Bridged, Resistor_THT:R_Axial_DIN0204_L3.6mm_D1.6mm_P5.08mm_Horizontal, F.Cu at (156.8, 77.9)
- moved DRV1 28.8 mm to (113.1, 97.3)
- moved Motor1 26.3 mm to (114.9, 84.7), turned to 180 degrees
- moved PowerSupply1 9.62 mm to (115.1, 71.5), turned to 180 degrees
Connections:
- net Net-(DRV1-In1) renamed /In1
- net Net-(DRV1-In2) renamed /In2
Routing:
- net /In2: track 84.3 -> 131.8 mm
- net /In1: track 79.7 -> 102.4 mm
- net GND: track 145.9 -> 165.0 mm
- net Net-(DRV1-PW_+): track 10.2 -> 29.0 mm
- net Net-(DRV1-Out_1): track 9.22 -> 20.6 mm
- net Net-(DRV1-Out_2): track 8.82 -> 13.9 mm
Other:
- board size 95.6 x 65 mm -> 90 x 57.8 mm

Commit message: Final PCB Update (For Now)
Other:
- board size 90 x 57.8 mm -> 90 x 59.5 mm
Changed lines of the file:
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@@
 	)
 	(gr_rect
-		(start 100.74 66.5)
+		(start 100.74 64.86)
 		(end 190.69 124.32)
 		(stroke
@@
 		(polygon
 			(pts
-				(xy 100.728664 66.49) (xy 190.74 65.936193) (xy 190.67 123.43) (xy 190.63 123.51) (xy 101.11 124.26)
+				(xy 100.720865 65.309342) (xy 190.741436 64.755478) (xy 190.67 123.43) (xy 190.63 123.51) (xy 101.11 124.26)
 			)
 		)
