File: Hardware/PCBModels/ArduinoShieldDesign/CEWBPCBDesign.kicad_sch (KiCad schematic)
At the start: 6 parts

Commit message: Updated PCB Design
Parts:
- added JP1, JP2: Jumper_2_Bridged, Resistor_THT:R_Axial_DIN0204_L3.6mm_D1.6mm_P5.08mm_Horizontal, symbol Jumper:Jumper_2_Bridged
Connections:
- net In2: now reaches A1.D10, DRV1.1 (In2)
- net In2: now also JP2.1 (A), JP2.2 (B)
- net In1: now reaches A1.D9, DRV1.2 (In1)
- net In1: now also JP1.1 (A), JP1.2 (B)

Commit message: Final PCB Update (For Now)
Other:
- moved on the sheet: JP2
Changed lines of the file:
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@@
 	)
 	(junction
-		(at 118.11 134.62)
+		(at 114.3 133.35)
 		(diameter 0)
 		(color 0 0 0 0)
@@
 	(wire
 		(pts
-			(xy 116.84 134.62) (xy 118.11 134.62)
+			(xy 113.03 133.35) (xy 114.3 133.35)
 		)
 		(stroke
@@
 	(wire
 		(pts
-			(xy 129.54 139.7) (xy 118.11 139.7)
+			(xy 125.73 138.43) (xy 114.3 138.43)
 		)
 		(stroke
@@
 	(wire
 		(pts
-			(xy 118.11 139.7) (xy 118.11 134.62)
-		)
-		(stroke
-			(width 0)
-			(type default)
-		)
-	)
-	(wire
-		(pts
-			(xy 118.11 134.62) (xy 119.38 134.62)
+			(xy 114.3 138.43) (xy 114.3 133.35)
+		)
+		(stroke
+			(width 0)
+			(type default)
+		)
+	)
+	(wire
+		(pts
+			(xy 114.3 133.35) (xy 115.57 133.35)
 		)
 		(stroke
@@
 	(wire
 		(pts
-			(xy 129.54 134.62) (xy 129.54 139.7)
+			(xy 125.73 133.35) (xy 125.73 138.43)
 		)
 		(stroke
@@
 	)
 	(label "In2"
-		(at 116.84 134.62 180)
+		(at 113.03 133.35 180)
 		(effects
 			(font
@@
 	(symbol
 		(lib_id "Jumper:Jumper_2_Bridged")
-		(at 124.46 134.62 0)
+		(at 120.65 133.35 0)
 		(unit 1)
 		(exclude_from_sim no)
@@
 		(dnp no)
 		(property "Reference" "JP2"
-			(at 124.46 129.54 0)
+			(at 120.65 128.27 0)
 			(effects
 				(font
@@
 		)
 		(property "Value" "Jumper_2_Bridged"
-			(at 124.46 132.08 0)
+			(at 120.65 130.81 0)
 			(effects
 				(font
@@
 		)
 		(property "Footprint" "Resistor_THT:R_Axial_DIN0204_L3.6mm_D1.6mm_P5.08mm_Horizontal"
-			(at 124.46 134.62 0)
+			(at 120.65 133.35 0)
 			(effects
 				(font
@@
 		)
 		(property "Datasheet" "~"
-			(at 124.46 134.62 0)
+			(at 120.65 133.35 0)
 			(effects
 				(font
@@
 		)
 		(property "Description" "Jumper, 2-pole, closed/bridged"
-			(at 124.46 134.62 0)
-			(effects
-				(font
+			(at 120.65 133.35 0)
+			(effects
+				(font
