File: Hardware/PCBModels/ArduinoShieldDesign/ForwardDesign/ForwardCEWBPCBDesign.kicad_sch (KiCad schematic)
At the start: 8 parts

Commit message: Adding Images and Cleaning up
Connections:
- net +5C: no longer JP4.1 (A), JP4.2 (B), MainEncoder1.1 (Pin_1), SecondaryEncoder1.1 (Pin_1)
- new net +5V: JP4.1 (A), JP4.2 (B), MainEncoder1.1 (Pin_1), SecondaryEncoder1.1 (Pin_1)
Changed lines of the file:
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@@
 			)
 		)
-		(property "Value" "+5C"
+		(property "Value" "+5V"
 			(at 156.21 54.61 0)
 			(effects
@@
 			)
 		)
-		(property "Value" "+5C"
+		(property "Value" "+5V"
 			(at 113.03 54.61 0)
 			(effects
